Commit message: refactor: Change my_gokart structure
Add 6 casters to support my_gokart model

File: catkin_ws/src/my_gokart/urdf/my_gokart.xacro (robot description, xacro)
@@ -10,5 +10,5 @@
     <pose>0 0 0.1 0 0 0</pose>
     <inertial>
-      <mass value="15.0"/>
+      <mass value="30.0"/>
       <origin xyz="0.0 0 0" rpy=" 0 0 0"/>
       <inertia
@@ -31,5 +31,5 @@
     </visual>
     <collision name='front_left_caster_collision'>
-      <origin xyz="1.9 .4 -0.05" rpy=" 0 0 0"/>
+      <origin xyz="0.9 .35 -0.05" rpy=" 0 0 0"/>
       <geometry>
         <sphere radius="0.0499"/>
@@ -37,5 +37,65 @@
     </collision>
     <visual name='front_left_caster_visual'>
-      <origin xyz="1.9 .4 -0.05" rpy=" 0 0 0"/>
+      <origin xyz="0.9 .35 -0.05" rpy=" 0 0 0"/>
+      <geometry>
+        <sphere radius="0.05"/>
+      </geometry>
+    </visual>
+    <collision name='front_right_caster_collision'>
+      <origin xyz="0.9 -0.35 -0.05" rpy=" 0 0 0"/>
+      <geometry>
+        <sphere radius="0.0499"/>
+      </geometry>
+    </collision>
+    <visual name='front_right_caster_visual'>
+      <origin xyz="0.9 -0.35 -0.05" rpy=" 0 0 0"/>
+      <geometry>
+        <sphere radius="0.05"/>
+      </geometry>
+    </visual>
+    <collision name='center_left_caster_collision'>
+      <origin xyz="0 0.35 -0.05" rpy=" 0 0 0"/>
+      <geometry>
+        <sphere radius="0.0499"/>
+      </geometry>
+    </collision>
+    <visual name='center_left_caster_visual'>
+      <origin xyz="0 0.35 -0.05" rpy=" 0 0 0"/>
+      <geometry>
+        <sphere radius="0.05"/>
+      </geometry>
+    </visual>
+    <collision name='center_right_caster_collision'>
+      <origin xyz="0 -0.35 -0.05" rpy=" 0 0 0"/>
+      <geometry>
+        <sphere radius="0.0499"/>
+      </geometry>
+    </collision>
+    <visual name='center_right_caster_visual'>
+      <origin xyz="0 -0.35 -0.05" rpy=" 0 0 0"/>
+      <geometry>
+        <sphere radius="0.05"/>
+      </geometry>
+    </visual>
+    <collision name='rear_left_caster_collision'>
+      <origin xyz="-0.9 0.35 -0.05" rpy=" 0 0 0"/>
+      <geometry>
+        <sphere radius="0.0499"/>
+      </geometry>
+    </collision>
+    <visual name='rear_left_caster_visual'>
+      <origin xyz="-0.9 0.35 -0.05" rpy=" 0 0 0"/>
+      <geometry>
+        <sphere radius="0.05"/>
+      </geometry>
+    </visual>
+    <collision name='rear_right_caster_collision'>
+      <origin xyz="-0.9 -0.35 -0.05" rpy=" 0 0 0"/>
+      <geometry>
+        <sphere radius="0.0499"/>
+      </geometry>
+    </collision>
+    <visual name='rear_right_caster_visual'>
+      <origin xyz="-0.9 -0.35 -0.05" rpy=" 0 0 0"/>
       <geometry>
         <sphere radius="0.05"/>

Commit message: refactor: Change my_gokart model and plugin
Change my_gokart model and plugin for 4 wheels

File: catkin_ws/src/my_gokart/urdf/my_gokart.xacro (robot description, xacro)
@@ -2,4 +2,5 @@
 <robot name="my_gokart" xmlns:xacro="http://www.ros.org/wiki/xacro">
   <link name="robot_footprint"></link>
+  <xacro:include filename="$(find my_gokart)/urdf/my_gokart.gazebo" />
   <joint name="robot_footprint_joint" type="fixed">
     <origin xyz="0 0 0" rpy="0 0 0" />
@@ -10,5 +11,5 @@
     <pose>0 0 0.1 0 0 0</pose>
     <inertial>
-      <mass value="30.0"/>
+      <mass value="50.0"/>
       <origin xyz="0.0 0 0" rpy=" 0 0 0"/>
       <inertia
@@ -30,4 +31,16 @@
       </geometry>
     </visual>
+    <collision name='sensor_platform_collision'>
+      <origin xyz="0.8 0 0.1" rpy=" 0 0 0"/>
+      <geometry>
+        <box size=".1 .1 .3"/>
+      </geometry>
+    </collision>
+    <visual name='sensor_platform_visual'>
+      <origin xyz="0.8 0 0.1" rpy=" 0 0 0"/>
+      <geometry>
+        <box size=".1 .1 .3"/>
+      </geometry>
+    </visual>
     <collision name='front_left_caster_collision'>
       <origin xyz="0.9 .35 -0.05" rpy=" 0 0 0"/>
@@ -103,3 +116,195 @@
     </visual>
   </link>
+  <link name='front_left_wheel'>
+    <pose>0 0 0 0 0 0</pose>
+    <inertial>
+      <mass value="5.0"/>
+      <origin xyz="0.0 0 0" rpy=" 0 1.5707 1.5707"/>
+      <inertia
+          ixx="0.1" ixy="0" ixz="0"
+          iyy="0.1" iyz="0"
+          izz="0.1"
+      />
+    </inertial>
+    <collision name='front_left_wheel_collision'>
+      <origin xyz="0 0 0" rpy=" 0 1.5707 1.5707"/>
+      <geometry>
+        <cylinder radius="0.14" length="0.21"/>
+      </geometry>
+    </collision>
+    <visual name='front_left_wheel_visual'>
+      <origin xyz="0 0 0" rpy=" 0 1.5707 1.5707"/>
+      <geometry>
+        <cylinder radius="0.14" length="0.21"/>
+      </geometry>
+    </visual>
+  </link>
+  <link name='front_right_wheel'>
+    <pose>0 0 0 0 0 0</pose>
+    <inertial>
+      <mass value="5.0"/>
+      <origin xyz="0.0 0 0" rpy=" 0 1.5707 1.5707"/>
+      <inertia
+          ixx="0.1" ixy="0" ixz="0"
+          iyy="0.1" iyz="0"
+          izz="0.1"
+      />
+    </inertial>
+    <collision name='front_right_wheel_collision'>
+      <origin xyz="0 0 0" rpy=" 0 1.5707 1.5707"/>
+      <geometry>
+        <cylinder radius="0.14" length="0.21"/>
+      </geometry>
+    </collision>
+    <visual name='front_right_wheel_visual'>
+      <origin xyz="0 0 0" rpy=" 0 1.5707 1.5707"/>
+      <geometry>
+        <cylinder radius="0.14" length="0.21"/>
+      </geometry>
+    </visual>
+  </link>
+  <link name='rear_left_wheel'>
+    <pose>0 0 0 0 0 0</pose>
+    <inertial>
+      <mass value="5.0"/>
+      <origin xyz="0.0 0 0" rpy=" 0 1.5707 1.5707"/>
+      <inertia
+          ixx="0.1" ixy="0" ixz="0"
+          iyy="0.1" iyz="0"
+          izz="0.1"
+      />
+    </inertial>
+    <collision name='rear_left_wheel_collision'>
+      <origin xyz="0 0 0" rpy=" 0 1.5707 1.5707"/>
+      <geometry>
+        <cylinder radius="0.14" length="0.21"/>
+      </geometry>
+    </collision>
+    <visual name='rear_left_wheel_visual'>
+      <origin xyz="0 0 0" rpy=" 0 1.5707 1.5707"/>
+      <geometry>
+        <cylinder radius="0.14" length="0.21"/>
+      </geometry>
+    </visual>
+  </link>
+  <link name='rear_right_wheel'>
+    <pose>0 0 0 0 0 0</pose>
+    <inertial>
+      <mass value="5.0"/>
+      <origin xyz="0.0 0 0" rpy=" 0 1.5707 1.5707"/>
+      <inertia
+          ixx="0.1" ixy="0" ixz="0"
+          iyy="0.1" iyz="0"
+          izz="0.1"
+      />
+    </inertial>
+    <collision name='rear_right_wheel_collision'>
+      <origin xyz="0 0 0" rpy=" 0 1.5707 1.5707"/>
+      <geometry>
+        <cylinder radius="0.14" length="0.21"/>
+      </geometry>
+    </collision>
+    <visual name='rear_right_wheel_visual'>
+      <origin xyz="0 0 0" rpy=" 0 1.5707 1.5707"/>
+      <geometry>
+        <cylinder radius="0.14" length="0.21"/>
+      </geometry>
+    </visual>
+  </link>
+  <joint type="continuous" name="front_left_wheel_hinge">
+    <origin xyz="0.9 0.6 0" rpy="0 0 0"/>
+    <child link="front_left_wheel"/>
+    <parent link="chassis"/>
+    <axis xyz="0 1 0" rpy="0 0 0"/>
+    <limit effort="10000" velocity="1000"/>
+    <dynamics damping="1.0" friction="1.0"/>
+  </joint>
+  <joint type="continuous" name="front_right_wheel_hinge">
+    <origin xyz="0.9 -0.6 0" rpy="0 0 0"/>
+    <child link="front_right_wheel"/>
+    <parent link="chassis"/>
+    <axis xyz="0 1 0" rpy="0 0 0"/>
+    <limit effort="10000" velocity="1000"/>
+    <dynamics damping="1.0" friction="1.0"/>
+  </joint>
+  <joint type="continuous" name="rear_left_wheel_hinge">
+    <origin xyz="-0.9 0.6 0" rpy="0 0 0"/>
+    <child link="rear_left_wheel"/>
+    <parent link="chassis"/>
+    <axis xyz="0 1 0" rpy="0 0 0"/>
+    <limit effort="10000" velocity="1000"/>
+    <dynamics damping="1.0" friction="1.0"/>
+  </joint>
+  <joint type="continuous" name="rear_right_wheel_hinge">
+    <origin xyz="-0.9 -0.6 0" rpy="0 0 0"/>
+    <child link="rear_right_wheel"/>
+    <parent link="chassis"/>
+    <axis xyz="0 1 0" rpy="0 0 0"/>
+    <limit effort="10000" velocity="1000"/>
+    <dynamics damping="1.0" friction="1.0"/>
+  </joint>
+  <link name='camera'>
+    <pose>0 0 0 0 0 0</pose>
+    <inertial>
+      <mass value="0.1"/>
+      <origin xyz="0.0 0 0" rpy="0.0 0 0"/>
+      <inertia
+          ixx="1e-6" ixy="0" ixz="0"
+          iyy="1e-6" iyz="0"
+          izz="1e-6"
+      />
+    </inertial>
+    <collision name='collision'>
+      <origin xyz="0 0 0" rpy=" 0 0 0"/>
+      <geometry>
+        <box size="0.05 0.05 0.05"/>
+      </geometry>
+    </collision>
+    <visual name='camera_visual'>
+      <origin xyz="0 0 0" rpy="0 0 0"/>
+      <geometry>
+        <box size="0.05 0.05 0.05"/>
+      </geometry>
+    </visual>
+  </link>
+  <joint type="fixed" name="camera_joint">
+    <origin xyz="1.0 0 0" rpy="0 0 0"/>
+    <child link="camera"/>
+    <parent link="chassis"/>
+    <axis xyz="0 1 0" rpy="0 0 0"/>
+    <limit effort="10000" velocity="1000"/>
+    <dynamics damping="1.0" friction="1.0"/>
+  </joint>
+  <link name='hokuyo'>
+    <pose>0 0 0 0 0 0</pose>
+    <inertial>
+      <mass value="1e-5"/>
+      <origin xyz="0.0 0 0" rpy="0.0 0 0"/>
+      <inertia
+          ixx="1e-6" ixy="0" ixz="0"
+          iyy="1e-6" iyz="0"
+          izz="1e-6"
+      />
+    </inertial>
+    <collision name='collision'>
+      <origin xyz="0 0 0" rpy=" 0 0 0"/>
+      <geometry>
+        <box size="0.1 0.1 0.1"/>
+      </geometry>
+    </collision>
+    <visual name='hokuyo_visual'>
+      <origin xyz="0 0 0" rpy="0 0 0"/>
+      <geometry>
+        <mesh filename="package://my_robot/meshes/hokuyo.dae"/>
+      </geometry>
+    </visual>
+  </link>
+  <joint type="fixed" name="hokuyo_joint">
+    <origin xyz="0.8 0.0 0.3" rpy="0 0 0"/>
+    <child link="hokuyo"/>
+    <parent link="chassis"/>
+    <axis xyz="0 1 0" rpy="0 0 0"/>
+    <limit effort="10000" velocity="1000"/>
+    <dynamics damping="1.0" friction="1.0"/>
+  </joint>
 </robot>

Commit message: refactor: House my gokart in my office
House my gokart in my office
Lower mass of my gokart so it doesn't spin

File: catkin_ws/src/my_gokart/urdf/my_gokart.xacro (robot description, xacro)
@@ -11,5 +11,5 @@
     <pose>0 0 0.1 0 0 0</pose>
     <inertial>
-      <mass value="50.0"/>
+      <mass value="10.0"/>
       <origin xyz="0.0 0 0" rpy=" 0 0 0"/>
       <inertia
